Commit message: 修改：     controllers/wbc/TaskContact/LinkPosTask.cpp 	修改：     controllers/wbc_config.yaml 	修改：     estimate/estimate.cpp 	修改：     estimate/state.h 	修改：     h1_description/mjcf/h1.xml 	修改：     h1_description/mjcf/h1_arm_fixed.xml 	修改：     h1_description/mjcf/h1_leg_fixed.xml 	修改：     h1_description/mjcf/h1_torso_fixed.xml 	修改：     h1_description/urdf/h1_left_arm.urdf 	修改：     h1_description/urdf/h1_left_leg.urdf 	修改：     h1_description/urdf/h1_right_arm.urdf 	修改：     h1_description/urdf/h1_right_leg.urdf 	修改：     main.cpp 	修改：     test/FSM.cpp 	修改：     test/motion_planning/motion_planning.cpp 	修改：     utils/dynamics.cpp 	修改：     utils/kinematics.cpp 	修改：     utils/kinematics.h

File: h1_description/urdf/h1_left_arm.urdf (robot description, URDF)
Before this commit: robot h1_description, 7 links, 6 joints
Links:
- added link world
Joints:
- added joint floating_base_joint: type floating, parent world, child pelvis

File: h1_description/urdf/h1_left_leg.urdf (robot description, URDF)
Before this commit: robot h1_description, 9 links, 8 joints
Links:
- added link world
Joints:
- added joint floating_base_joint: type floating, parent world, child pelvis

File: h1_description/urdf/h1_right_arm.urdf (robot description, URDF)
Before this commit: robot h1_description, 7 links, 6 joints
Links:
- added link world
Joints:
- added joint floating_base_joint: type floating, parent world, child pelvis

File: h1_description/urdf/h1_right_leg.urdf (robot description, URDF)
Before this commit: robot h1_description, 9 links, 8 joints
Links:
- added link world
Joints:
- added joint floating_base_joint: type floating, parent world, child pelvis
