Commit message: 修改：     controllers/wbc/TaskContact/LinkPosTask.cpp 	修改：     controllers/wbc_config.yaml 	修改：     estimate/estimate.cpp 	新文件：   h1_description/mjcf/h1.xml 	修改：     h1_description/mjcf/h1_leg_fixed.xml 	修改：     h1_description/mjcf/scene.xml 	修改：     h1_description/urdf/h1.urdf 	修改：     h1_description/urdf/h1_left_arm.urdf 	修改：     h1_description/urdf/h1_right_arm.urdf 	修改：     test/FSM.cpp 	修改：     utils/dynamics.cpp 	修改：     utils/dynamics.hpp

File: h1_description/urdf/h1.urdf (robot description, URDF)
Before this commit: robot h1_description, 29 links, 28 joints
Links:
- added link left_hand_center
- added link right_hand_center
Joints:
- added joint left_hand_center_joint: type fixed, parent left_elbow_link, child left_hand_center, origin xyz=0.2605 0 -0.0185 rpy=0 0 0
- added joint right_hand_center_joint: type fixed, parent right_elbow_link, child right_hand_center, origin xyz=0.2605 0 -0.0185 rpy=0 0 0

File: h1_description/urdf/h1_left_arm.urdf (robot description, URDF)
Before this commit: robot h1_description, 6 links, 5 joints
Links:
- added link left_hand_center
Joints:
- added joint left_hand_center_joint: type fixed, parent left_elbow_link, child left_hand_center, origin xyz=0.2605 0 -0.0185 rpy=0 0 0

File: h1_description/urdf/h1_right_arm.urdf (robot description, URDF)
Before this commit: robot h1_description, 6 links, 5 joints
Links:
- added link right_hand_center
Joints:
- added joint right_hand_center_joint: type fixed, parent right_elbow_link, child right_hand_center, origin xyz=0.2605 0 -0.0185 rpy=0 0 0

Commit message: 修改：     controllers/mpc/mpc_caller.cpp 	修改：     controllers/mpc_config.yaml 	修改：     controllers/wbc/DynWbc.cpp 	新文件：   controllers/wbc/TaskContact/ArmPosTask.cpp 	重命名：   controllers/wbc/TaskContact/LinkPosTask.hpp -> controllers/wbc/TaskContact/ArmPosTask.hpp 	修改：     controllers/wbc/TaskContact/BodyOriTask.cpp 	修改：     controllers/wbc/TaskContact/BodyPosTask.cpp 	重命名：   controllers/wbc/TaskContact/LinkPosTask.cpp -> controllers/wbc/TaskContact/LegPosTask.cpp 	新文件：   controllers/wbc/TaskContact/LegPosTask.hpp 	修改：     controllers/wbc/TaskContact/SingleContact.cpp 	修改：     controllers/wbc/WbcCtrl.cpp 	修改：     controllers/wbc/WbcCtrl.hpp 	修改：     controllers/wbc_config.yaml 	修改：     estimate/estimate.cpp 	修改：     estimate/state.h 	修改：     h1_description/mjcf/h1_arm_fixed.xml 	修改：     h1_description/mjcf/h1_leg_fixed.xml 	修改：     h1_description/mjcf/h1_torso_fixed.xml 	修改：     h1_description/mjcf/scene.xml 	修改：     h1_description/urdf/h1.urdf 	修改：     h1_description/urdf/h1_left_arm.urdf 	修改：     h1_description/urdf/h1_right_arm.urdf 	修改：     main.cpp 	修改：     test/FSM.cpp 	修改：     test/FSM.h 	修改：     test/demo/demo_container.cpp 	修改：     test/motion_planning/motion_planning.cpp 	修改：     utils/cppTypes.h 	修改：     utils/dynamics.cpp 	修改：     utils/dynamics.hpp 	修改：     utils/kinematics.cpp 	修改：     utils/kinematics.h

File: h1_description/urdf/h1.urdf (robot description, URDF)
Before this commit: robot h1_description, 31 links, 30 joints
Joints:
- joint torso_joint: limit lower=-2.35 upper=2.35 effort=200 velocity=23 -> (none); type revolute -> fixed

File: h1_description/urdf/h1_left_arm.urdf (robot description, URDF)
Before this commit: robot h1_description, 8 links, 7 joints
Joints:
- joint torso_joint: limit lower=-2.35 upper=2.35 effort=200 velocity=23 -> (none); type revolute -> fixed

File: h1_description/urdf/h1_right_arm.urdf (robot description, URDF)
Before this commit: robot h1_description, 8 links, 7 joints
Joints:
- joint torso_joint: limit lower=-2.35 upper=2.35 effort=200 velocity=23 -> (none); type revolute -> fixed
